File: Hardware/proiect.sch (EAGLE design)
At the start: 105 parts, among them IC1 BQ25180YBGR, IC2 DRV2605YZFR, IC3 BMA421, IC9 RT6160AWSC, J1 503480-2400, J2 TC2030-IDC_TC2030-IDC, J4 KH-TYPE-C-16P, Q1 20V/4.2A/52mΩ/1.4W, Q3 \SI1308EDL-T1-GE3, U1 NRF52840_QF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

Commit message: update sch
Parts:
- IC3: value BMA421 -> BMA423
- L1: value 3.9pH -> 3.9nH
- R1, R_PWR_EPD: device InkTime_v5:ERA-1AEB3401C_CPF0201D7K68C1 -> InkTime_v5:CPF0201D7K68C1_CPF0201D7K68C1
Connections:
- net N$30 renamed P0.26
- net N$31 renamed P0.27
- net N$32 renamed P0.04
- net N$33 renamed EPD_CS/2.2D
- net N$38 renamed P1.09
- net N$42 renamed HAPTIC_EN/2.6A
- removed net N$34: U1.P0.06@L1
- removed net N$35: U1.P0.07@M2
- removed net N$36: U1.P0.08@N1
- removed net N$37: U1.P1.08@P2
- removed net N$39: U1.P0.11@T2
- removed net N$44: C6.1, U1.VDD@W1, U1.VDDH@Y2
- removed net PREBGL: EPD_C11.2, J1.23
- removed net SC/1.4C: IC2.SCL
- net 3V3/2.4A: now also C6.1, U1.VDD@W1, U1.VDDH@Y2
- net IMU_INT1: now also U1.P0.08@N1
- net IMU_INT2: now also U1.P1.08@P2
- net PMIC_INT: now also U1.P0.11@T2
- net PREVGL: now also EPD_C11.2, J1.23
- net SCL/1.4C: now also IC2.SCL
- net SCL/2.4C: now also U1.P0.07@M2
- net SDA/2.4C: now also U1.P0.06@L1
